File: aps_radar/transmitter.sch (KiCad schematic (older format))
At the start: 0 parts

Commit message: Began transmitter layout
Parts:
- added C?: 1uF, symbol Device:C_Small
- added C? (x2): 0.1uF, symbol Device:C_Small
- added JP?: OSC_EN, symbol Device:Jumper_NO_Small
- added R? (x3): 18, symbol Device:R_Small
- added R? (x2): 68, symbol Device:R_Small
- added U?: LMX2491RTWR, RTW0024A, symbol aps_radar_lib:LMX2491RTWR
- added Y?: CWX813, symbol aps_radar_lib:CWX813
Connections:
- new net: JP?.2, Y?.1 (EN)
- new net: R?.2, Y?.3 (OUT)
- new net: C?.2, U?.10 (GND_OSCIN*)
- new net: C?.2, U?.9 (OSCIN)
- new net: R?.1, R?.1, R?.2
- new net: C?.1, R?.1 (x2)
- new net: R?.2, R?.2
- new net +3V3: C?.1, Y?.4 (VCC)
- new net GND: U?.1 (GND), U?.11 (GND), U?.2 (GND), U?.25 (PAD), U?.3 (GND)
- new net VCC: U?.18 (VCC), U?.19 (VCC), U?.6 (VCC), U?.7 (VCC), U?.8 (VCC)
Other:
- note added: "Disable"
- note added: "Enable"
- note added: "High / Open"
- note added: "Low"
- note added: "→"
